File: hardware/canbus-outpost/canbus-outpost.kicad_sch (KiCad schematic)
At the start: 117 parts, among them J1 SERVO, J10 RJ45, J11 SWD, J12 UART, J13 RJ45, J14 GPIO, J2 DCC_SIG, J3 BOOSTER, J4 TRACK1, J5 TRACK2, J6 TRACK3, J7 TRACK4, J8 VDC, J9 USB, SW1 BUTTON, SW2 BUTTON, U1 W25Q32JVSS, U10 ISO7720D, U11 L78L05_SO8, U12 ISO7720D, U13 ISO7720D, U14 ISO7720D, U2 RP2350A, U3 TPS5430DDA, U4 SN65HVD230, U5 XC6206PxxxMR, U6 LM393, U7 LM393, U8 LM393, U9 LM393, Y1 ABM8-272-T3

Commit message: fix: update part rotations
Parts:
- U10, U11, U12, U13, U14: JLCPCB_CORRECTION (none) -> 0;0;-90
Changed lines of the file:
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@@
 			)
 		)
+		(property "JLCPCB_CORRECTION" "0;0;-90"
+			(at 243.84 74.93 0)
+			(effects
+				(font
+					(size 1.27 1.27)
+				)
+				(hide yes)
+			)
+		)
 		(pin "2"
 		)
@@
 			)
 		)
+		(property "JLCPCB_CORRECTION" "0;0;-90"
+			(at 328.93 43.18 0)
+			(effects
+				(font
+					(size 1.27 1.27)
+				)
+				(hide yes)
+			)
+		)
 		(pin "5"
 		)
@@
 			)
 		)
+		(property "JLCPCB_CORRECTION" "0;0;-90"
+			(at 243.84 134.62 0)
+			(effects
+				(font
+					(size 1.27 1.27)
+				)
+				(hide yes)
+			)
+		)
 		(pin "2"
 		)
@@
 			)
 		)
+		(property "JLCPCB_CORRECTION" "0;0;-90"
+			(at 243.84 166.37 0)
+			(effects
+				(font
+					(size 1.27 1.27)
+				)
+				(hide yes)
+			)
+		)
 		(pin "2"
 		)
@@
 			(at 243.84 106.68 0)
 			(effects
+				(font
+					(size 1.27 1.27)
+				)
+				(hide yes)
+			)
+		)
+		(property "JLCPCB_CORRECTION" "0;0;-90"
+			(at 243.84 106.68 0)
+			(effects

Commit message: fix: switch from LM393 to TLV3202 for railcom signals
Parts:
- U6, U7, U8, U9: value LM393 -> TLV3202; LCSC C7955 -> C129325
Changed lines of the file:
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@@
 			)
 		)
-		(property "Value" "LM393"
+		(property "Value" "TLV3202"
 			(at 373.38 125.73 0)
 			(effects
@@
 			)
 		)
-		(property "LCSC" "C7955"
+		(property "LCSC" "C129325"
 			(at 373.38 118.11 0)
 			(effects
@@
 			)
 		)
-		(property "Value" "LM393"
+		(property "Value" "TLV3202"
 			(at 373.38 181.61 0)
 			(effects
@@
 			)
 		)
-		(property "LCSC" "C7955"
+		(property "LCSC" "C129325"
 			(at 373.38 173.99 0)
 			(effects
@@
 			)
 		)
-		(property "Value" "LM393"
+		(property "Value" "TLV3202"
 			(at 373.888 153.67 0)
 			(effects
@@
 			)
 		)
-		(property "LCSC" "C7955"
+		(property "LCSC" "C129325"
 			(at 373.38 147.32 0)
 			(effects
@@
 			)
 		)
-		(property "Value" "LM393"
+		(property "Value" "TLV3202"
 			(at 373.888 97.79 0)
 			(effects
@@
 			)
 		)
-		(property "LCSC" "C7955"
+		(property "LCSC" "C129325"
 			(at 373.38 91.44 0)
 			(effects
@@
 			)
 		)
-		(property "Value" "LM393"
+		(property "Value" "TLV3202"
 			(at 373.38 69.85 0)
 			(effects
@@
 			)
 		)
-		(property "LCSC" "C7955"
+		(property "LCSC" "C129325"
 			(at 373.38 62.23 0)
 			(effects
@@
 			)
 		)
-		(property "Value" "LM393"
+		(property "Value" "TLV3202"
 			(at 377.19 142.748 0)
 			(effects
@@
 			)
 		)
-		(property "LCSC" "C7955"
+		(property "LCSC" "C129325"
 			(at 373.38 147.32 0)
 			(effects
@@
 			)
 		)
-		(property "Value" "LM393"
+		(property "Value" "TLV3202"
 			(at 377.19 198.628 0)
 			(effects
@@
 			)
 		)
-		(property "LCSC" "C7955"
+		(property "LCSC" "C129325"
 			(at 373.38 203.2 0)
 			(effects
@@
 			)
 		)
-		(property "Value" "LM393"
+		(property "Value" "TLV3202"
 			(at 377.19 86.868 0)
 			(effects
@@
 			)
 		)
-		(property "LCSC" "C7955"
+		(property "LCSC" "C129325"
 			(at 373.38 91.44 0)
 			(effects
@@
 			)
 		)
-		(property "Value" "LM393"
+		(property "Value" "TLV3202"
 			(at 377.19 30.988 0)
 			(effects
@@
 			)
 		)
-		(property "LCSC" "C7955"
+		(property "LCSC" "C129325"
 			(at 373.38 35.56 0)
 			(effects
@@
 			)
 		)
-		(property "Value" "LM393"
+		(property "Value" "TLV3202"
 			(at 373.888 41.91 0)
 			(effects
@@
 			)
 		)
-		(property "LCSC" "C7955"
+		(property "LCSC" "C129325"
 			(at 373.38 35.56 0)
 			(effects
@@
 			)
 		)
-		(property "Value" "LM393"
+		(property "Value" "TLV3202"
 			(at 373.38 237.49 0)
 			(effects
@@
 			)
 		)
-		(property "LCSC" "C7955"
+		(property "LCSC" "C129325"
 			(at 373.38 229.87 0)
 			(effects
@@
 			)
 		)
-		(property "Value" "LM393"
+		(property "Value" "TLV3202"
 			(at 373.888 209.55 0)
 			(effects
@@
 			)
 		)
-		(property "LCSC" "C7955"
+		(property "LCSC" "C129325"
 			(at 373.38 203.2 0)
 			(effects
