File: hardware/canbus-outpost/canbus-outpost.kicad_pcb (KiCad board)
At the start: 2 copper layers, 48 x 90 mm, 151 parts, among them J1 SERVO, J10 RJ45, J11 SWD, J12 UART, J13 RJ45, J14 GPIO, J2 DCC_SIG, J3 BOOSTER, J4 TRACK1, J5 TRACK2, J6 TRACK3, J7 TRACK4, J8 VDC, J9 USB, SW1 BUTTON, SW2 BUTTON, U1 W25Q32JVSS, U10 ISO7720D, U11 L78L05_SO8, U12 ISO7720D, U13 ISO7720D, U14 ISO7720D, U2 RP2350A, U3 TPS5430DDA, U4 SN65HVD230, U5 XC6206PxxxMR, U6 LM393, U7 LM393, U8 LM393, U9 LM393, Y1 ABM8-272-T3

Commit message: fix(hardware): fix railcom circuits
Parts:
- removed C24: 100uF, Library:CP_Elec_6.3x7.7
- removed D4: SS54, Library:D_SMA
- removed J12: UART, Library:PinHeader_1x03_P2.54mm_Vertical
- removed R12, R13: 220R, Library:R_0402_1005Metric
- removed R22, R23, R24, R25, R26, R27, R28, R29: 10K, Library:R_0402_1005Metric
- removed kibuzzard-688B6FED: G***, kibuzzard-688B6FED
- removed kibuzzard-688B7E7A: G***, kibuzzard-688B7E7A
- removed kibuzzard-688BED1C: G***, kibuzzard-688BED1C
- removed kibuzzard-688BF02A: G***, kibuzzard-688BF02A
- removed kibuzzard-688BF068: G***, kibuzzard-688BF068
- removed kibuzzard-688BF06D: G***, kibuzzard-688BF06D
- removed kibuzzard-688BF073: G***, kibuzzard-688BF073
- removed kibuzzard-688BF123: G***, kibuzzard-688BF123
- removed kibuzzard-688D37F3: G***, kibuzzard-688D37F3
- removed kibuzzard-688D37FE: G***, kibuzzard-688D37FE
- removed kibuzzard-688D3808: G***, kibuzzard-688D3808
- added C35: 100nF, Library:C_0402_1005Metric, F.Cu at (128.5, 89.5)
- added C36: 100nF, Library:C_0402_1005Metric, B.Cu at (151.5, 78.1)
- added C37: 100nF, Library:C_0402_1005Metric, B.Cu at (151.5, 87.6)
- added C38: 100nF, Library:C_0402_1005Metric, B.Cu at (151.5, 97.2)
- added C39: 100nF, Library:C_0402_1005Metric, B.Cu at (151.5, 106.6)
- added R31: 1K, Library:R_0402_1005Metric, F.Cu at (157.2, 79.1)
- added R32: 1K, Library:R_0402_1005Metric, F.Cu at (157.1, 88.6)
- added R33: 1K, Library:R_0402_1005Metric, F.Cu at (157.1, 98.1)
- added R34: 1K, Library:R_0402_1005Metric, F.Cu at (157.2, 107.5)
- added R35: 2.2K, Library:R_1206_3216Metric, F.Cu at (147.9, 52.4)
- added R36: 4.7K, Library:R_0402_1005Metric, F.Cu at (140.6, 85.3)
- added R37: 1K, Library:R_0402_1005Metric, B.Cu at (150.1, 90.0)
- added R38: 330K, Library:R_0402_1005Metric, B.Cu at (150.1, 91.0)
- added R39: 1K, Library:R_0402_1005Metric, B.Cu at (150.1, 99.4)
- added R40: 330K, Library:R_0402_1005Metric, B.Cu at (150.1, 100.3)
- added R41: 1K, Library:R_0402_1005Metric, B.Cu at (150.1, 70.9)
- added R42: 330K, Library:R_0402_1005Metric, B.Cu at (150.1, 71.9)
- added U15: TLP290(GB-TP,SE), Package_SO:SOIC-4_4.55x2.6mm_P1.27mm, B.Cu at (141.5, 65.7)
- added kibuzzard-69DC490B: G***, kibuzzard-69DC490B, F.Cu at (122.4, 88.9)
- added kibuzzard-69DC4912: G***, kibuzzard-69DC4912, F.Cu at (122.4, 91.4)
- added kibuzzard-69DC4921: G***, kibuzzard-69DC4921, F.Cu at (122.4, 94.0)
- added kibuzzard-69DC492A: G***, kibuzzard-69DC492A, F.Cu at (122.4, 96.5)
- added kibuzzard-69DC4DF3: G***, kibuzzard-69DC4DF3, F.Cu at (122.4, 99.1)
- added kibuzzard-69DC4DFC: G***, kibuzzard-69DC4DFC, F.Cu at (122.4, 101.6)
- added kibuzzard-69DC4E03: G***, kibuzzard-69DC4E03, F.Cu at (122.4, 104.2)
- added kibuzzard-69DC4E0F: G***, kibuzzard-69DC4E0F, F.Cu at (122.4, 106.8)
- C23: value 100uF -> 100nF; footprint Library:CP_Elec_6.3x7.7 -> Library:C_0402_1005Metric; moved to B.Cu
- D5: value SS54 -> 1N5819WS; footprint Library:D_SMA -> Diode_SMD:D_SOD-323
- J14: footprint Library:PinHeader_1x04_P2.54mm_Vertical -> Connector_PinHeader_2.54mm:PinHeader_1x08_P2.54mm_Vertical
- J4: value TRACK1 -> TRACK4
- J5: value TRACK2 -> TRACK3
- J6: value TRACK3 -> TRACK2
- J7: value TRACK4 -> TRACK1
- R11, R30: value 220R -> 1K
- R14: value 270K -> 330K
- R15: moved to B.Cu
- R16: value 820R -> 330K; moved to B.Cu
- R17: value 33K -> 1K; moved to B.Cu
- U6, U7, U8, U9: value LM393 -> TLV3202
- moved R15 32.5 mm to (154.5, 87.7)
- moved C23 27.8 mm to (154.5, 88.6)
- moved R16 26.5 mm to (150.1, 81.4), turned to 0 degrees
- moved R17 26.5 mm to (150.1, 80.4), turned to 180 degrees
- moved D5 20.5 mm to (138.3, 71.7), turned to 90 degrees
- moved kibuzzard-688B7D39 10.4 mm to (131.1, 96.3)
- moved J11 6.57 mm to (128.6, 93.8)
- moved kibuzzard-688BEEB4 6.57 mm to (131.5, 93.8)
- moved kibuzzard-688BF0B8 6.57 mm to (131.5, 98.9)
- moved kibuzzard-688BF0BD 6.57 mm to (131.5, 96.3)
- moved C1 6.44 mm to (133.0, 74.8), turned to -90 degrees
- moved J14 2.94 mm to (125.4, 88.9)
- moved J9 2.06 mm to (135.6, 71.9)
- moved kibuzzard-688BF1D4 2.06 mm to (131.8, 69.8)
- moved NT1 1.39 mm to (151.0, 107.0)
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Connections:
- C23 pad 1: /BOOSTER_R -> /RC_REF_H
- C23 pad 2: Net-(C23-Pad2) -> /BOOSTER_R
- D5 pad 1: GNDA -> +5V
- D5 pad 2: /BOOSTER_R -> Net-(D5-A)
- J9 pad 1: +5V -> Net-(D5-A)
- R14 pad 2: /RC_REF_L -> /RC_REF_H
- R15 pad 1: /RC_REF_L -> /RC_REF_H
- R16 pad 1: /BOOSTER_R -> +5VR
- R16 pad 2: /RC_REF_H -> Net-(U7A--)
- R17 pad 1: /RC_REF_H -> /TRACK_R3
- R17 pad 2: GNDA -> Net-(U7A--)
- U2 pad 12: unconnected-(U2-GPIO8-Pad12) -> /GPIO8
- U2 pad 13: unconnected-(U2-GPIO9-Pad13) -> /GPIO9
- U2 pad 14: unconnected-(U2-GPIO10-Pad14) -> /GPIO10
- U2 pad 15: unconnected-(U2-GPIO11-Pad15) -> /GPIO11
- U2 pad 43: unconnected-(U2-GPIO29_ADC3-Pad43) -> /CUTOUT_SIGNAL
- U4 pad 6: /CAN_H -> /CAN_L
- U4 pad 7: /CAN_L -> /CAN_H
- U6 pad 2: /TRACK_R4 -> Net-(U6A--)
- U6 pad 3: /RC_REF_H -> /BOOSTER_R
- U6 pad 4: GNDA -> /BOOSTER_R
- U6 pad 5: /TRACK_R4 -> Net-(U6B-+)
- U6 pad 6: /RC_REF_L -> /RC_REF_H
- U7 pad 2: /TRACK_R3 -> Net-(U7A--)
- U7 pad 3: /RC_REF_H -> /BOOSTER_R
- U7 pad 4: GNDA -> /BOOSTER_R
- U7 pad 5: /TRACK_R3 -> Net-(U7B-+)
- U7 pad 6: /RC_REF_L -> /RC_REF_H
- U8 pad 2: /TRACK_R2 -> Net-(U8A--)
- U8 pad 3: /RC_REF_H -> /BOOSTER_R
- U8 pad 4: GNDA -> /BOOSTER_R
- U8 pad 5: /TRACK_R2 -> Net-(U8B-+)
- U8 pad 6: /RC_REF_L -> /RC_REF_H
- U9 pad 2: /TRACK_R1 -> Net-(U9A--)
- U9 pad 3: /RC_REF_H -> /BOOSTER_R
- U9 pad 4: GNDA -> /BOOSTER_R
- U9 pad 5: /TRACK_R1 -> Net-(U9B-+)
- U9 pad 6: /RC_REF_L -> /RC_REF_H
Routing:
- net /RC_REF_L: track 56.0 -> 0.00 mm, vias 1 -> 0
- net +3.3V: track 100.9 -> 53.7 mm, vias 8 -> 18
- net /CUTOUT_SIGNAL: track 0.00 -> 25.8 mm, vias 0 -> 1
- net GNDA: track 25.0 -> 0.00 mm, vias 1 -> 0
- net Net-(D4-A): track 21.9 -> 0.00 mm
- net Net-(R35-Pad1): track 0.00 -> 20.9 mm, vias 0 -> 1
- net /GPIO11: track 0.00 -> 20.0 mm, vias 0 -> 1
- net /GPIO10: track 0.00 -> 17.9 mm, vias 0 -> 1
- net GND: track 14.1 -> 31.1 mm, vias 41 -> 58
- net /GPIO9: track 0.00 -> 15.8 mm, vias 0 -> 1
- net Net-(C23-Pad2): track 14.0 -> 0.00 mm, vias 2 -> 0
- net /RX: track 13.8 -> 0.00 mm
- net /GPIO8: track 0.00 -> 13.7 mm, vias 0 -> 1
- net /BOOSTER_L: track 48.7 -> 39.3 mm
- net +5V: track 78.9 -> 88.1 mm, vias 1 -> 4
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- added copper zone on In2.Cu, net +3.3V
- added copper zone on B.Cu, net /BOOSTER_R
- added copper zone on In1.Cu, net /CAN_GND
- added copper zone on In1.Cu, net GND
- added copper zone on In2.Cu, net VDC
- removed copper zone on F.Cu, net /CAN_GND
- removed copper zone on B.Cu, net GNDA
Other:
- copper layers 2 -> 4
- board text added: "CAN BUS OUTPOST"
- board text removed: "CANBUS OUTPOST"

Commit message: feat: add usb jack for flashing
Parts:
- removed kibuzzard-688BF1D4: G***, kibuzzard-688BF1D4
- added R12: 5.1K, Library:R_0402_1005Metric, F.Cu at (127.2, 74.2)
- added R13: 5.1K, Library:R_0402_1005Metric, F.Cu at (127.2, 75.2)
- J9: footprint Library:PinHeader_1x04_P2.54mm_Vertical -> Connector_USB:USB_C_Receptacle_GCT_USB4115-03-C
- moved SW1 11.7 mm to (123.0, 72.7)
- moved kibuzzard-688BEB22 11.7 mm to (125.4, 72.7)
- moved C1 10.6 mm to (122.5, 76.2), turned to 180 degrees
- moved R2 5.86 mm to (122.5, 86.5)
- moved U1 5.77 mm to (124.5, 81.4), turned to 90 degrees
- moved J9 5.14 mm to (131.3, 74.8)
- moved D5 1.79 mm to (136.8, 72.6), turned to 180 degrees
Routing:
- net Net-(R2-Pad2): track 5.49 -> 16.3 mm
- net Net-(D5-A): track 3.26 -> 11.7 mm, vias 0 -> 2
- net Net-(J9-CC1): track 0.00 -> 7.78 mm, vias 0 -> 2
- net /QSPI_SD3: track 10.9 -> 16.3 mm
- net /QSPI_SCLK: track 9.27 -> 14.2 mm
- net /QSPI_SD0: track 6.63 -> 10.3 mm
- net /QSPI_CS: track 17.7 -> 14.1 mm
- net /QSPI_SD1: track 16.3 -> 13.1 mm
- net Net-(J9-CC2): track 0.00 -> 3.00 mm
- net +3.3V: track 53.7 -> 56.7 mm, vias 18 -> 16
- net /D-: track 10.9 -> 8.97 mm
- net /D+: track 10.9 -> 12.2 mm, vias 0 -> 3
- net /QSPI_SD2: track 12.0 -> 10.8 mm
- net GND: track 31.1 -> 32.2 mm

Commit message: feat: add SSSB LED signal header
Parts:
- added C24: 100nF, Library:C_0402_1005Metric, F.Cu at (137.1, 105.7)
- added F2: 750mA, Fuse:Fuse_1206_3216Metric, F.Cu at (139.6, 105.0)
- added J12: GND, Connector_PinHeader_2.54mm:PinHeader_1x02_P2.54mm_Vertical, F.Cu at (128.7, 104.1)
- added J15: LIGHTS, Library:PinHeader_1x03_P2.54mm_Vertical, F.Cu at (137.0, 108.9)
- added R22: 33R, Library:R_0402_1005Metric, F.Cu at (136.1, 105.7)
- added U16: 74AHCT1G125, Package_TO_SOT_SMD:SOT-23-5, F.Cu at (136.7, 102.2)
- added kibuzzard-6AE53D03: G***, kibuzzard-6AE53D03, F.Cu at (129.1, 101.8)
- added kibuzzard-6AE558B7: G***, kibuzzard-6AE558B7, F.Cu at (139.2, 111.2)
Connections:
- U2 pad 42: unconnected-(U2-GPIO28_ADC2-Pad42) -> /LIGHTS
Routing:
- net /LIGHTS: track 0.00 -> 18.9 mm, vias 0 -> 2
- net +5V: track 88.1 -> 93.2 mm, vias 4 -> 5
- net Net-(J15-Pin_1): track 0.00 -> 3.09 mm
- net Net-(J15-Pin_2): track 0.00 -> 2.57 mm
- net Net-(R22-Pad1): track 0.00 -> 2.03 mm
- net GNDD: track 58.8 -> 58.3 mm, vias 2 -> 0
- net GND: track 32.2 -> 32.1 mm, vias 58 -> 61
